Commit message: update jdamr_cube.urdf to move arm and wheels forward to improve balance and reach.

File: jdamr_cube_description/urdf/jdamr_cube2.urdf (robot description, URDF)
Before this commit: robot jdamr_cube, 17 links, 16 joints
Joints:
- joint arm_riser_joint: origin xyz=0.12 0 0.075 rpy=0 0 0 -> xyz=0 0 0.075 rpy=0 0 0
- joint left_wheel_joint: origin xyz=0.15 0.175 -0.008 rpy=0 0 0 -> xyz=0 0.175 -0.008 rpy=0 0 0
- joint right_wheel_joint: origin xyz=0.15 -0.175 -0.008 rpy=0 0 0 -> xyz=0 -0.175 -0.008 rpy=0 0 0
