Commit message: fix(description): 그리퍼 손가락 충돌 지오메트리 정밀화 및 RGBD 카메라 각도 조정
- 손가락 충돌을 STL 메쉬 실측 기반 primitive 박스 6개로 교체 (트라이메시 관통 해결)
- 손끝에 가상 패드 확장 적용 (실물 고무 패드 근사, 강체 파지 성립)
- RGBD 카메라 pitch 0.9→0.45로 완화 (서 있는 물체 원거리 검출 가능)

Co-Authored-By: Claude Fable 5 <noreply@anthropic.com>

File: jdamr_cube_description/urdf/jdamr_cube.urdf (robot description, URDF)
Before this commit: robot jdamr_cube, 19 links, 18 joints
Links:
- link arm_gripper_link: geometry collision box size=0.0229 0.0243 0.0299; collision box size=0.0286 0.0238 0.0319
- link arm_moving_jaw_link: geometry collision box size=0.0181 0.0129 0.0203; collision box size=0.0200 0.0399 0.0480
Joints:
- joint rgbd_camera_joint: origin xyz=0.05 0 0.4 rpy=0 0.9 0 -> xyz=0.05 0 0.4 rpy=0 0.45 0

Commit message: fix(description): 그리퍼 고정 죠 가상 패드 제거, STL 실측 충돌 복원
Co-Authored-By: Claude Fable 5 <noreply@anthropic.com>

File: jdamr_cube_description/urdf/jdamr_cube.urdf (robot description, URDF)
Before this commit: robot jdamr_cube, 19 links, 18 joints
Links:
- link arm_gripper_link: geometry collision box size=0.0156 0.0158 0.0299; collision box size=0.0229 0.0243 0.0299

Commit message: feat(capstone_pick): 쓰레기통 투입 + 파지 판정·캘리브레이션 정밀화
쓰레기통 투입 (실제 투입 실증: 큐브가 개구부 중앙 3cm 이내 착지)
- 회색 통 검출: 무채색(S<45)+어두움(45<V<115)+뎁스·높이 게이트. 뎁스 상한을 넓히면
  원경 벽이 통과 한 덩어리로 붙어 통째로 기각되므로 2.0m 유지
- 통 중심 추정은 뎁스 앞면에 반깊이(0.08) 보정, 근접 락으로 마스크 편향 회피
  (통이 화면을 채우면 중심이 한쪽 벽으로 치우쳐 방위가 수렴하지 않음)
- 역투영 높이 게이트를 대상별로 분리 (물체 0.20 / 통 0.60)

파지 판정 (가짜 성공 제거)
- 각도 구간 판정(0.05~0.45): 하한만 두면 미닫힘(0.0)이 성공으로 새고,
  명령 대비 잔여각으로 보면 재조임이 목표에 도달하는 순간 오판
- holding()은 살짝 더 조여보는 능동 확인 — 물체가 빠져도 그리퍼는 직전 명령 위치를
  유지하므로 각도만으로는 낙하를 잡지 못함. 파지 실패 시 운반·투입으로 넘어가지 않음

캘리브레이션·제어 정정
- 파지 포켓 0.361→0.381 (스윕 실측: 0.361은 하강이 큐브를 3.5mm 밀어냄, 0.381은 밀림 0)
- 손목캠 기준·게인을 새 포켓에서 직접 실측 (환산값은 46px 어긋나 정렬이 모서리로 수렴)
  pan 게인은 pan을 실제로 돌려 잰 값 사용 — 물체 이동 환산은 카메라 동반 회전이 빠져 진동
- move_arm이 관절 실도달을 확인 (궤적 시간이 끝나면 못 따라온 채 완료되어 다음 명령과
  겹치며 급가속 발생)
- 손가락 마찰·접촉 강성을 고무 패드 수준으로, 그리퍼 조인트 effort 한계 10→25

Co-Authored-By: Claude Fable 5 <noreply@anthropic.com>

File: jdamr_cube_description/urdf/jdamr_cube.urdf (robot description, URDF)
Before this commit: robot jdamr_cube, 19 links, 18 joints
Links:
- link arm_gripper_link: geometry collision box size=0.0196 0.0188 0.0309; collision box size=0.0229 0.0243 0.0299
Joints:
- joint arm_gripper: limit lower=-0.174533 upper=1.74533 effort=10 velocity=10 -> lower=-0.174533 upper=1.74533 effort=25 velocity=10

Commit message: fix(capstone_pick): 파지 실패 회귀 복구 — 파지력·마찰 강화가 역효과였음
들기까지 포함한 포켓 스윕으로 원인 특정: 실물 근사라며 넣은 설정들이 강체 시뮬에서
오히려 물체를 튕겨내 어느 포켓에서도 큐브가 바닥을 떠나지 못했다.
- 그리퍼 조인트 effort 25→10, 명령 effort 20→10 복원
- 손가락 마찰·접촉 강성(mu/kp/kd/minDepth) 태그 제거
- 손끝 패드 제거(STL 실측 복원) — 5mm·3mm 모두 들기 실패, 원래 값에서만 성공
- 검증: 포켓 0.361/0.376/0.391 세 곳 모두 LIFTED(z 0.169~0.172), 옆에 놓기 E2E 성공

손목캠 pan 게인 1740→1277 (호버 자세에서 pan을 직접 돌려 실측, 이전 값은 과대라
보정이 매번 부족했음), 정렬 임계 0.012→0.006rad, 반복 4→6회

Co-Authored-By: Claude Fable 5 <noreply@anthropic.com>

File: jdamr_cube_description/urdf/jdamr_cube.urdf (robot description, URDF)
Before this commit: robot jdamr_cube, 19 links, 18 joints
Links:
- link arm_gripper_link: geometry collision box size=0.0156 0.0158 0.0299; collision box size=0.0229 0.0243 0.0299
Joints:
- joint arm_gripper: limit lower=-0.174533 upper=1.74533 effort=25 velocity=10 -> lower=-0.174533 upper=1.74533 effort=10 velocity=10

Commit message: revert(description/tools): 접촉 물성 커스텀 초기화 — 공식 SO-101 상태로
르로봇 시연 데이터 기반 파지로 전환하기 위해 손가락 충돌 박스 6개,
gazebo 마찰 태그(μ·minDepth), 큐브 비틀림 마찰·μ 상향을 모두 제거하고
공식 URDF의 메시 충돌·기본 물성으로 되돌린다.

Co-Authored-By: Claude Opus 5 (1M context) <noreply@anthropic.com>

File: jdamr_cube_description/urdf/jdamr_cube.urdf (robot description, URDF)
Before this commit: robot jdamr_cube, 19 links, 18 joints
Links:
- link arm_gripper_link: geometry collision mesh filename=package://jdamr_cube_description/meshes/so101/sts3215_03a_v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; collision mesh filename=package://jdamr_cube_description/meshes/so101/wrist_roll_fo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
- link arm_moving_jaw_link: geometry collision mesh filename=package://jdamr_cube_description/meshes/so101/moving_jaw_so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; visual mesh filename=package://jdamr_cube_description/meshes/so101/moving_jaw_so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

Commit message: feat(tools): LeRobot 시연 데이터 재생 파이프라인 — 시뮬 파지 성립
svla_so101_pickplace 시연을 우리 시뮬에서 재생해 파지를 성립시켰다
(ep0: 들림 +49mm, 운반 53mm, 스톨각 -0.082 물림 확인, 실좌표 판정).
우리 팔 URDF가 공식 so101_new_calib와 관절 단위로 동일함을 대조 확인했고,
정규화 액션(-100~100)을 공식 한계로 라디안 매핑한 것이 정합의 근거다.

- lerobot_extract.py: 데이터셋 → 라디안 궤적 npy (conda lerobot 환경)
- lerobot_replay.py: 자가 캘리브레이션 2패스 — 정적 FK 프로브로 닫힘
  프레임의 핀치 좌표·닫힘 방향을 측정(재생 중 측정은 gz 서브프로세스
  지연으로 17cm 표류 — 실측), 그 좌표에 시연 제원 레고(2x4, 2.5g)와
  넓은 테이블을 놓고 재생. 판정은 백그라운드 z 추적(들림)+실좌표
- 손가락 충돌 박스 복원: 공식 STL 메시 충돌만으로는 죠가 물체를 관통해
  어떤 방식으로도 파지가 성립하지 않는다(재확인) — 마찰 튜닝 없이
  기하 수정만 유지
- stop_stack.sh: 시뮬 유닛은 세션 종료 후에도 상시 CPU를 태운다(팬 폭주
  실사례) — 작업 종료 시 필수 실행

함정 기록: 질량 0 가상 링크는 gz에서 병합돼 베이스 좌표라는 허수를
반환한다. 링크 자세는 모델 상대다(모델 자세와 합성 필요). 엔티티
제거는 비동기라 동명 재생성 전 소멸 폴링이 필요하다.

Co-Authored-By: Claude Opus 5 (1M context) <noreply@anthropic.com>

File: jdamr_cube_description/urdf/jdamr_cube.urdf (robot description, URDF)
Before this commit: robot jdamr_cube, 19 links, 18 joints
Links:
- link arm_gripper_link: geometry collision box size=0.0156 0.0158 0.0299; collision box size=0.0229 0.0243 0.0299
- link arm_moving_jaw_link: geometry collision box size=0.0181 0.0129 0.0203; collision box size=0.0200 0.0399 0.0480

Commit message: fix(sim/tools): 관통 파지 제거 — 정직한 접촉 + 고무 근사로 진짜 파지 성립
사용자 관찰로 드러난 결함: 시연 닫힘 명령(-0.14)은 레고 폭을 한참 지나친
목표라 위치 제어가 손가락을 관통시켜, 레고가 그리퍼에 '꽂힌 채' 운반되는
가짜 성공이 양산됐다(49편 수집분 무효 처리).

- 그리퍼 닫힘 클램프 -0.035 + effort 5: 실물의 접촉 스톨 재현(관통 불가)
- 스톨각 지속 캡처 + pinch_ok(-0.06~+0.08) 판정을 성공 조건에 결합 —
  관통(-0.1 이하)과 진짜 물림이 라벨로 갈린다
- 손가락 μ6·minDepth + 레고 비틀림 마찰 복원: 정직한 접촉에서 운반 미끄럼을
  잡는 물리(들림 후 낙하 반복 → 재도입 근거 실측)
- 차체 밸러스트 3→15kg: 팔 반동에 차체가 들리고 비주행 방향으로 틀어지던
  것 해소(사용자 요구, 재생 후 rpy 0 근방 실측)
- 관측 카메라 재배치: up은 테이블 직상공(작업 영역 중심), side는 작업
  영역 중앙 — 시연 구도 정합(마스트·섀시 가림 제거)
- 대시보드 현행화: 관측 상공·측면·손목 3뷰

검증(ep19): 들림 +58mm, 운반 74mm, success=True, 스톨 -0.035 진짜 물림.

Co-Authored-By: Claude Opus 5 (1M context) <noreply@anthropic.com>

File: jdamr_cube_description/urdf/jdamr_cube.urdf (robot description, URDF)
Before this commit: robot jdamr_cube, 19 links, 18 joints
Links:
- link base_link: mass 3.0 -> 15.0

Commit message: feat(teleop): 웹 조종기(WASD·터치)와 라이다 실측 반영
web_teleop: 파이 8080 포트에서 브라우저 WASD·폰 터치로 cmd_vel,
3중 데드맨(킵얼라이브→신선도→펌웨어 워치독), 정지 확정 후 침묵해
다른 발행자와 공존. 브링업은 LD14P·230400 실측 반영, URDF 는 바퀴축
원점 정합과 라이다 실측 오프셋(전방 7.5cm·좌 2cm) 적용.

Co-Authored-By: Claude Fable 5 <noreply@anthropic.com>

File: jdamr_cube_description/urdf/jdamr_cube.urdf (robot description, URDF)
Before this commit: robot jdamr_cube, 19 links, 18 joints
Joints:
- joint laser_joint: origin xyz=0.25 0 0.1 rpy=0 0 0 -> xyz=0.075 0.02 0.1 rpy=0 0 0
- joint left_wheel_joint: origin xyz=0.15 0.175 -0.008 rpy=0 0 0 -> xyz=0 0.175 -0.008 rpy=0 0 0
- joint right_wheel_joint: origin xyz=0.15 -0.175 -0.008 rpy=0 0 0 -> xyz=0 -0.175 -0.008 rpy=0 0 0

Commit message: fix(slam): 실측 4건 반영 — 라이다 후방 장착·타임스탬프 지연·상관매칭 오프
사진 판독으로 라이다가 축 후방 7.5cm 임을 확정(부호 반전, 15cm 오류
제거)하고 차체를 실물 정사각 비례로. ldlidar 드라이버가 한 바퀴 수신
완료 시각을 시작 시각으로 찍던 버그를 규약대로 보정(회전 중 ~6도
왜곡 원인). 복도 세로축 점프를 만드는 전역 상관매칭을 끄고 캘리브
레이션된 오도메트리를 씨앗으로 쓴다. joint_state_publisher 포함.
※ 파이 오프라인으로 재빌드·실지도 검증은 미완 — 다음 가동 시 배포.

Co-Authored-By: Claude Fable 5 <noreply@anthropic.com>

File: jdamr_cube_description/urdf/jdamr_cube.urdf (robot description, URDF)
Before this commit: robot jdamr_cube, 19 links, 18 joints
Links:
- link base_link: geometry collision box size=0.18 0.18 0.12; visual box size=0.18 0.18 0.12
Joints:
- joint laser_joint: origin xyz=0.075 0.02 0.1 rpy=0 0 0 -> xyz=-0.075 0.02 0.1 rpy=0 0 0

Commit message: fix(slam): 거울반전 제거와 라이다 오프셋 실측 반영 — 지도 붕괴의 진짜 원인
laser_scan_dir 을 8/14 에 False 로 뒤집은 것이 오류였다. 로봇이 CCW 로
+θ 돌면 로봇 좌표계에서 세상은 −θ 도는 것이 정상인데, 자작 프로브가
그 −θ 를 거울반전으로 오판해 멀쩡한 스캔에 거울을 씌웠다. 실물 확인:
오른쪽 코너가 지도에서 왼쪽에 그려짐. 이후 나흘간의 지도 꼬임과 매칭
튜닝(max_range·상관매칭·가중치)이 전부 이 잘못된 전제 위에 있었다.

라이다 위치도 사진 판독값(후방 75mm)이 오류였다 — 줄자 실측은 전방
40mm·좌 55mm 로, 115mm 어긋난 채 회전마다 스캔이 공전하고 있었다.

수정 후 실측: 확신 벽 5.49%(정상 대역 2~6%), 상단 벽이 한 겹으로
이어지고 직각 코너 확보, 겹침 소멸.

Co-Authored-By: Claude Opus 5 (1M context) <noreply@anthropic.com>

File: jdamr_cube_description/urdf/jdamr_cube.urdf (robot description, URDF)
Before this commit: robot jdamr_cube, 19 links, 18 joints
Joints:
- joint laser_joint: origin xyz=-0.075 0.02 0.1 rpy=0 0 0 -> xyz=0.04 0.055 0.1 rpy=0 0 0
