Commit message: updated the jdamr_cube_description package to include the new so101 robot model, including its meshes, URDF, and controller configuration. Also updated the Gazebo launch file and package.xml to support the new model.

File: jdamr_cube_description/urdf/jdamr_cube.urdf (robot description, URDF)
Before this commit: robot jdamr_cube, 7 links, 6 joints
Links:
- added link arm_base_link, mass 0.147; collision mesh filename=package://jdamr_cube_description/meshes/so101/base_motor_ho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; collision mesh filename=package://jdamr_cube_description/meshes/so101/base_so101_v2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
- added link arm_gripper_frame_link, mass 1e-9
- added link arm_gripper_link, mass 0.087; collision mesh filename=package://jdamr_cube_description/meshes/so101/sts3215_03a_v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; collision mesh filename=package://jdamr_cube_description/meshes/so101/wrist_roll_fo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
- added link arm_lower_arm_link, mass 0.104; collision mesh filename=package://jdamr_cube_description/meshes/so101/motor_holder_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; collision mesh filename=package://jdamr_cube_description/meshes/so101/sts3215_03a_v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
- added link arm_moving_jaw_link, mass 0.012; collision mesh filename=package://jdamr_cube_description/meshes/so101/moving_jaw_so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; visual mesh filename=package://jdamr_cube_description/meshes/so101/moving_jaw_so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
- added link arm_shoulder_link, mass 0.100006; collision mesh filename=package://jdamr_cube_description/meshes/so101/motor_holder_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; collision mesh filename=package://jdamr_cube_description/meshes/so101/rotation_pitc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
- added link arm_upper_arm_link, mass 0.103; collision mesh filename=package://jdamr_cube_description/meshes/so101/sts3215_03a_v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; collision mesh filename=package://jdamr_cube_description/meshes/so101/upper_arm_so1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
- added link arm_wrist_link, mass 0.079; collision mesh filename=package://jdamr_cube_description/meshes/so101/sts3215_03a_n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; collision mesh filename=package://jdamr_cube_description/meshes/so101/wrist_roll_pi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
Joints:
- added joint arm_elbow_flex: type revolute, parent arm_upper_arm_link, child arm_lower_arm_link, origin xyz=-0.11257 -0.028 1.73763e-16 rpy=-3.63608e-16 8.74301e-16 1.5708, axis 0 0 1, limit lower=-1.69 upper=1.69 effort=10 velocity=10
- added joint arm_gripper: type revolute, parent arm_gripper_link, child arm_moving_jaw_link, origin xyz=0.0202 0.0188 -0.0234 rpy=1.5708 -5.24284e-08 -1.41553e-15, axis 0 0 1, limit lower=-0.174533 upper=1.74533 effort=10 velocity=10
- added joint arm_gripper_frame_joint: type fixed, parent arm_gripper_link, child arm_gripper_frame_link, origin xyz=-0.0079 -0.000218121 -0.0981274 rpy=0 3.14159 0
- added joint arm_mount_joint: type fixed, parent base_link, child arm_base_link, origin xyz=0 0 0.075 rpy=0 0 0
- added joint arm_shoulder_lift: type revolute, parent arm_shoulder_link, child arm_upper_arm_link, origin xyz=-0.0303992 -0.0182778 -0.0542 rpy=-1.5708 -1.5708 0, axis 0 0 1, limit lower=-1.74533 upper=1.74533 effort=10 velocity=10
- added joint arm_shoulder_pan: type revolute, parent arm_base_link, child arm_shoulder_link, origin xyz=0.0388353 -8.97657e-09 0.0624 rpy=3.14159 4.18253e-17 -3.14159, axis 0 0 1, limit lower=-1.91986 upper=1.91986 effort=10 velocity=10
- added joint arm_wrist_flex: type revolute, parent arm_lower_arm_link, child arm_wrist_link, origin xyz=-0.1349 0.0052 3.62355e-17 rpy=4.02456e-15 8.67362e-16 -1.5708, axis 0 0 1, limit lower=-1.65806 upper=1.65806 effort=10 velocity=10
- added joint arm_wrist_roll: type revolute, parent arm_wrist_link, child arm_gripper_link, origin xyz=5.55112e-17 -0.0611 0.0181 rpy=1.5708 0.0486795 3.14159, axis 0 0 1, limit lower=-2.74385 upper=2.84121 effort=10 velocity=10

Commit message: update arm_wrist_camera_link origin to avoid collision with arm itself in Nav2 collision_monitor.

File: jdamr_cube_description/urdf/jdamr_cube.urdf (robot description, URDF)
Before this commit: robot jdamr_cube, 15 links, 14 joints
Links:
- added link arm_riser_link, mass 0.05; collision box size=0.06 0.06 0.15; visual box size=0.06 0.06 0.15
- added link arm_wrist_camera_link, mass 0.005; collision box size=0.02 0.02 0.02; visual box size=0.02 0.02 0.02
Joints:
- added joint arm_riser_joint: type fixed, parent base_link, child arm_riser_link, origin xyz=0 0 0.075 rpy=0 0 0
- added joint arm_wrist_camera_joint: type fixed, parent arm_wrist_link, child arm_wrist_camera_link, origin xyz=0 -0.11 0.03 rpy=0 0 -1.5708
- joint arm_mount_joint: origin xyz=0 0 0.075 rpy=0 0 0 -> xyz=0 0 0.15 rpy=0 0 0; parent base_link -> arm_riser_link

Commit message: update joint_control.py to add --camera depth option for view command, and add colorize_depth() to visualize depth images. Update run_gazebo_slam.bat and run_navigation.bat to launch wrist, rgbd, and depth camera views.

File: jdamr_cube_description/urdf/jdamr_cube.urdf (robot description, URDF)
Before this commit: robot jdamr_cube, 17 links, 16 joints
Links:
- added link rgbd_camera_link, mass 0.02; collision box size=0.03 0.08 0.03; visual box size=0.03 0.08 0.03
- added link rgbd_mast_link, mass 0.05; collision box size=0.04 0.04 0.6; visual box size=0.04 0.04 0.6
Joints:
- added joint rgbd_camera_joint: type fixed, parent rgbd_mast_link, child rgbd_camera_link, origin xyz=0 0 0.6 rpy=0 0.7 0
- added joint rgbd_mast_joint: type fixed, parent base_link, child rgbd_mast_link, origin xyz=0 0 0.075 rpy=0 0 0

Commit message: updated:   jdamr_cube_so101_arm/jdamr_cube_so101_arm/joint_control.py

File: jdamr_cube_description/urdf/jdamr_cube.urdf (robot description, URDF)
Before this commit: robot jdamr_cube, 19 links, 18 joints
Joints:
- joint rgbd_camera_joint: origin xyz=0 0 0.6 rpy=0 0.7 0 -> xyz=0.05 0 0.6 rpy=0 0.9 0

Commit message: updated:   scripts/wsl_run_arm_control.sh

File: jdamr_cube_description/urdf/jdamr_cube.urdf (robot description, URDF)
Before this commit: robot jdamr_cube, 19 links, 18 joints
Links:
- link arm_riser_link: geometry collision box size=0.06 0.06 0.0; visual box size=0.06 0.06 0.0
- link rgbd_mast_link: geometry collision box size=0.04 0.04 0.4; visual box size=0.04 0.04 0.4
Joints:
- joint arm_mount_joint: origin xyz=0 0 0.15 rpy=0 0 0 -> xyz=0 0 0 rpy=0 0 0
- joint rgbd_camera_joint: origin xyz=0.05 0 0.6 rpy=0 0.9 0 -> xyz=0.05 0 0.4 rpy=0 0.9 0

Commit message: update joint_control.py: add --no-home-init option to skip home initialization at start

File: jdamr_cube_description/urdf/jdamr_cube.urdf (robot description, URDF)
Before this commit: robot jdamr_cube, 19 links, 18 joints
Joints:
- joint laser_joint: origin xyz=0.3 0 0.15 rpy=0 0 0 -> xyz=0.25 0 0.1 rpy=0 0 0

Commit message: fix(slam): G4 중앙 장착과 검증된 실기 브링업 적용

File: jdamr_cube_description/urdf/jdamr_cube.urdf (robot description, URDF)
Before this commit: robot jdamr_cube, 19 links, 18 joints
Links:
- link laser_link: mass 0.05 -> 0.214; geometry collision cylinder length=0.0412 radius=0.03615; visual cylinder length=0.0412 radius=0.03615
Joints:
- joint laser_joint: origin xyz=0.04 0.055 0.1 rpy=0 0 0 -> xyz=0 0 0.1 rpy=0 0 3.141592653589793

Commit message: feat(slam): 새 차체 실측 제원과 라이다 TF 반영

File: jdamr_cube_description/urdf/jdamr_cube.urdf (robot description, URDF)
Before this commit: robot jdamr_cube, 19 links, 18 joints
Joints:
- joint laser_joint: origin xyz=0 0 0.1 rpy=0 0 3.141592653589793 -> xyz=-0.010 0 0.075 rpy=0 0 3.141592653589793
