Commit message: fix(description): IMU 보드 방향을 주행 bag으로 정해 imu_link로 선언
보드는 z 아래·y 앞·x 왼쪽(roll 180°, yaw 90°)으로 달려 있는데 드라이버가
frame base_link로 내고 있었다. 9/15–16 bag 5개에서 자이로 z/바퀴 회전율
-0.966~-0.996, 보드 y/바퀴 전진 가속 +1.15~+1.25(상관 0.87–0.93)였다.
URDF imu_joint와 드라이버 imu_frame=imu_link, 근거는 new_base_geometry.yaml,
보정 대장 항목을 바꾼다. 축 판정은 imu_axes.py와 합성 신호 테스트로 남긴다.

Co-Authored-By: Claude Opus 5.5 (1M context) <noreply@anthropic.com>

File: jdamr_cube_description/urdf/new_base_real.urdf (robot description, URDF)
Before this commit: robot new_base_real, 11 links, 10 joints
Links:
- added link imu_link
Joints:
- added joint imu_joint: type fixed, parent base_link, child imu_link, origin xyz=0 0 0 rpy=3.141592653589793 0 1.5707963267948966
