Commit message: fix(camera): 상판 위 54cm 렌즈 높이를 실차에 반영

File: jdamr_cube_description/urdf/new_base_real.urdf (robot description, URDF)
Before this commit: robot new_base_real, 12 links, 11 joints
Links:
- added link camera_link; visual box size=0.040 0.165 0.048
- added link upper_tabletop_surface_frame
Joints:
- added joint camera_mount_joint: type fixed, parent upper_tabletop_surface_frame, child camera_link, origin xyz=-0.275 0 0.540 rpy=0.011934068034722573 0.41246669799099545 -0.0007507445375463481
- added joint upper_tabletop_surface_joint: type fixed, parent base_link, child upper_tabletop_surface_frame, origin xyz=0 0 0.720 rpy=0 0 0
